File: SensorPack_v1/CAN_Transceiver.kicad_sch (KiCad schematic)
At the start: 6 parts, among them U2 MCP2562-E-SN

Commit message: Featured out SensorPack_v1
Parts:
- C1: renamed from C8; symbol Device:C -> Capstone_Symbols:C; KiLib_Generator (none) -> SMD_2terminal_chip_molded
- CM1: footprint Extra_Footprints:CMChoke_2.6x1.2mm_HandSolder -> Capstone_Footprints:CMChoke_2.6x1.2mm_HandSolder; symbol Device:L_Ferrite_Coupled -> Capstone_Symbols:L_Ferrite_Coupled
- D1: symbol Device:D_TVS_Dual_AAC -> Capstone_Symbols:D_TVS_Dual_AAC; KiLib_Generator (none) -> package/gullwing
- R4: renamed from R2; symbol Device:R -> Capstone_Symbols:R; KiLib_Generator (none) -> SMD_2terminal_chip_molded
- R5: renamed from R3; symbol Device:R -> Capstone_Symbols:R; KiLib_Generator (none) -> SMD_2terminal_chip_molded
- U1: renamed from U2; symbol Interface_CAN_LIN:MCP2562-E-SN -> Capstone_Symbols:MCP2562-E-SN; KiLib_Generator (none) -> package/gullwing

Commit message: Final changes to Sensor Pack
Parts:
- R4, R5: Digikey Part (none) -> RMCF0603FT10R0
- U1: Digikey Part (none) -> MCP2562-E/SN
Other:
- company: (none) -> Vector Drive
- title: (none) -> Sensor Pack Board
Changed lines of the file:
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@@
 	(generator_version "10.0")
 	(paper "A4")
+	(title_block
+		(title "Sensor Pack Board")
+		(date "2026-09-24")
+		(rev "1.0")
+		(company "Vector Drive")
+		(comment 1 "By: Lucas Ngo")
+	)
 	(junction
 		(at 38.1 69.85)
@@
 			)
 		)
+		(property "Digikey Part" "MCP2562-E/SN"
+			(at 93.98 72.39 0)
+			(hide yes)
+			(show_name no)
+			(do_not_autoplace no)
+			(effects
+				(font
+					(size 1.27 1.27)
+				)
+			)
+		)
 		(pin "8"
 		)
@@
 			)
 		)
-		(property "Digikey Part" ""
+		(property "Digikey Part" "RMCF0603FT10R0"
 			(at 64.77 74.93 90)
 			(hide yes)
@@
 			)
 		)
-		(property "Digikey Part" ""
+		(property "Digikey Part" "RMCF0603FT10R0"
 			(at 64.77 69.85 90)
 			(hide yes)

Commit message: Tweaks
Parts:
- C1: Digikey Part CL10B104KB8NFNC -> CL10B104KO8NNNC
- D1: Digikey Part DESD12VL2BTQ-7 -> DESD15VL2BTQ-7
Changed lines of the file:
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@@
 			)
 		)
-		(property "Digikey Part" "CL10B104KB8NFNC"
+		(property "Digikey Part" "CL10B104KO8NNNC"
 			(at 88.9 53.34 0)
 			(hide yes)
@@
 			)
 		)
-		(property "Digikey Part" "DESD12VL2BTQ-7"
+		(property "Digikey Part" "DESD15VL2BTQ-7"
 			(at 46.99 85.09 0)
 			(hide yes)
