File: SensorPack_v1/SensorPack_v1.kicad_sch (KiCad schematic)
At the start: 25 parts, among them J2 M12x5 A-Type, J3 2x3 Header, J4 M12x5 A-Type, Q1 DMN2310U, U1 STM32C092KCT6, U4 TLV7xx_SOT23-5, Y1 8MHz 16pF Load

Commit message: Featured out SensorPack_v1
Parts:
- added J3, J4, J5, J6, J7, J9: 4p Header, Connector_PinHeader_2.54mm:PinHeader_1x04_P2.54mm_Vertical, symbol Capstone_Symbols:Conn_01x04_Pin
- added J8: 6p Header, Connector_PinHeader_2.54mm:PinHeader_1x06_P2.54mm_Vertical, symbol Capstone_Symbols:Conn_01x06_Pin
- added JP1, JP2, JP4, JP6: Jumper_3_Bridged12, Capstone_Footprints:Jumper_0603_2pos, symbol Capstone_Symbols:Jumper_3_Bridged12
- added JP3, JP5: Jumper_2_Small_Open, Resistor_SMD:R_0603_1608Metric_Pad0.98x0.95mm_HandSolder, symbol Capstone_Symbols:Jumper_2_Small_Open
- added R10, R14: 1k, Resistor_SMD:R_0603_1608Metric_Pad0.98x0.95mm_HandSolder, symbol Capstone_Symbols:R
- added R11, R15: 2k, Resistor_SMD:R_0603_1608Metric_Pad0.98x0.95mm_HandSolder, symbol Capstone_Symbols:R
- added R12, R13, R16, R17, R8, R9: 4k7, Resistor_SMD:R_0603_1608Metric_Pad0.98x0.95mm_HandSolder, symbol Capstone_Symbols:R
- C2: renamed from C1; symbol Device:C -> Capstone_Symbols:C; KiLib_Generator (none) -> SMD_2terminal_chip_molded
- C3: renamed from C2; symbol Device:C -> Capstone_Symbols:C; KiLib_Generator (none) -> SMD_2terminal_chip_molded
- C4: renamed from C3; symbol Device:C -> Capstone_Symbols:C; KiLib_Generator (none) -> SMD_2terminal_chip_molded
- C5: renamed from C12; symbol Device:C -> Capstone_Symbols:C; KiLib_Generator (none) -> SMD_2terminal_chip_molded
- C6: renamed from C9; symbol Device:C -> Capstone_Symbols:C; KiLib_Generator (none) -> SMD_2terminal_chip_molded
- C7: symbol Device:C -> Capstone_Symbols:C; KiLib_Generator (none) -> SMD_2terminal_chip_molded
- C8: renamed from C4; symbol Device:C -> Capstone_Symbols:C; KiLib_Generator (none) -> SMD_2terminal_chip_molded
- D2: renamed from D3; symbol Device:D_TVS -> Capstone_Symbols:D_TVS
- F1: symbol Device:Polyfuse -> Capstone_Symbols:Polyfuse; KiLib_Generator (none) -> SMD_2terminal_chip_molded
- FB1: symbol Device:FerriteBead -> Capstone_Symbols:FerriteBead; KiLib_Generator (none) -> SMD_2terminal_chip_molded
- J1: renamed from J2; footprint Extra_Footprints:M12x5_A_Circular_Connector -> Capstone_Footprints:M12x5_A_Circular_Connector; symbol Connector:Conn_01x05_Pin -> Capstone_Symbols:Conn_01x05_Pin
- J10: renamed from J3; value 2x3 Header -> 2x3 Pogo Header; footprint Extra_Footprints:2x03_2.54mm_DIP_pogo -> Capstone_Footprints:2x03_2.54mm_DIP_pogo; symbol Connector_Generic:Conn_02x03_Counter_Clockwise -> Capstone_Symbols:Conn_02x03_Counter_Clockwise
- J2: renamed from J4; footprint Extra_Footprints:M12x5_A_Circular_Connector -> Capstone_Footprints:M12x5_A_Circular_Connector; symbol Connector:Conn_01x05_Pin -> Capstone_Symbols:Conn_01x05_Pin
- LED1: footprint Connector_PinHeader_2.54mm:PinHeader_1x03_P2.54mm_Vertical -> LED_THT:LED_D3.0mm-3; symbol Device:LED_Dual_KAK -> Capstone_Symbols:LED_Dual_KAK; KiLib_Generator (none) -> connector/pin_header_socket
- Q1: symbol Transistor_FET:Q_NMOS_GSD -> Capstone_Symbols:Q_NMOS_GSD; KiLib_Generator (none) -> package/gullwing
- R1: renamed from R5; symbol Device:R -> Capstone_Symbols:R; KiLib_Generator (none) -> SMD_2terminal_chip_molded
- R2: renamed from R6; symbol Device:R -> Capstone_Symbols:R; KiLib_Generator (none) -> SMD_2terminal_chip_molded
- R3: renamed from R7; symbol Device:R -> Capstone_Symbols:R; KiLib_Generator (none) -> SMD_2terminal_chip_molded
- R6: renamed from R1; value 100k -> 10k; symbol Device:R -> Capstone_Symbols:R; KiLib_Generator (none) -> SMD_2terminal_chip_molded
- R7: renamed from R4; value 100k -> 10k; symbol Device:R -> Capstone_Symbols:R; KiLib_Generator (none) -> SMD_2terminal_chip_molded
- TH1: value NTC100k B3950 SMT -> NTC10k B3950 SMT; symbol Device:Thermistor_NTC -> Capstone_Symbols:Thermistor_NTC; KiLib_Generator (none) -> SMD_2terminal_chip_molded
- TH2: value NTC100k B3950 Probe -> NTC10k B3950 Probe; symbol Device:Thermistor_NTC -> Capstone_Symbols:Thermistor_NTC; KiLib_Generator (none) -> connector/pin_header_socket
- U2: renamed from U4; symbol Extra_Symbols:TLV7xx_SOT23-5 -> Capstone_Symbols:TLV7xx_SOT23-5; KiLib_Generator (none) -> package/gullwing
- U3: renamed from U1; symbol Local Symbols:STM32C092KCT6 -> Capstone_Symbols:STM32C092KCT6; KiLib_Generator (none) -> package/gullwing
- Y1: footprint Extra_Footprints:Crystal_6x3.5mm -> Capstone_Footprints:Crystal_6x3.5mm; symbol Device:Crystal -> Capstone_Symbols:Crystal
Connections:
- net +3V3: now also J4.2 (Pin_2), J6.2 (Pin_2), JP1.3 (B), JP2.3 (B), JP4.3 (B), JP6.3 (B), R12.1, R13.1, R16.1, R17.1, R8.1, R9.1
- net +5V: now also J4.1 (Pin_1), J6.1 (Pin_1), JP1.1 (A), JP2.1 (A), JP4.1 (A), JP6.1 (A)
- net GND: now also J3.2 (Pin_2), J4.3 (Pin_3), J5.2 (Pin_2), J6.3 (Pin_3), J7.2 (Pin_2), J8.2 (Pin_2), J9.1 (Pin_1), R11.2, R15.2
- net ADC_IN3: now reaches U3.10 (PA3)
- net ADC_IN3: now also JP5.2 (B), R14.2, R15.1
- net SPI1_CS1: now reaches U3.11 (PA4)
- net SPI1_CS1: now also J8.3 (Pin_3)
- net SPI1_SCK: now reaches U3.12 (PA5)
- net SPI1_SCK: now also J8.4 (Pin_4)
- net SPI1_MISO: now reaches U3.13 (PA6)
- net SPI1_MISO: now also J8.5 (Pin_5)
- net SPI1_MOSI: now reaches U3.14 (PA7)
- net SPI1_MOSI: now also J8.6 (Pin_6)
- net USART2_RX: now reaches U3.15 (PB0)
- net USART2_RX: now also J9.2 (Pin_2)
- net USART2_CK: now reaches U3.16 (PB1)
- net USART2_CK: now also J9.3 (Pin_3)
- net USART2_TX: now reaches U3.17 (PB2)
- net USART2_TX: now also J9.4 (Pin_4)
- net I2C1_SCL: now reaches U3.19 (PA9)
- net I2C1_SCL: now also J7.4 (Pin_4), R16.2
- net I2C1_SDA: now reaches U3.21 (PA10)
- net I2C1_SDA: now also J7.3 (Pin_3), R17.2
- net I2C2_SCL1: now reaches U3.22 (PA11[PA9])
- net I2C2_SCL1: now also J5.4 (Pin_4), R12.2
- net I2C2_SDA1: now reaches U3.23 (PA12[PA10])
- net I2C2_SDA1: now also J5.3 (Pin_3), R13.2
- net I2C2_SCL2: now reaches U3.27 (PB3)
- net I2C2_SCL2: now also J3.4 (Pin_4), R8.2
- net I2C2_SDA2: now reaches U3.28 (PB4)
- net I2C2_SDA2: now also J3.3 (Pin_3), R9.2
- net ADC_IN2: now reaches U3.9 (PA2)
- net ADC_IN2: now also JP3.2 (B), R10.2, R11.1
- new net: J4.4 (Pin_4), JP3.1 (A), R10.1
- new net: J3.1 (Pin_1), JP1.2 (C)
- new net: J8.1 (Pin_1), JP6.2 (C)
- new net: J5.1 (Pin_1), JP2.2 (C)
- new net: J6.4 (Pin_4), JP5.1 (A), R14.1
- new net: J7.1 (Pin_1), JP4.2 (C)
- no-connect marks 3 -> 6
Other:
- note added: "Analog input"
- note added: "Green"
- note added: "I2C Ports"
- note added: "Red"
- note added: "SPI Port"
- note added: "Sensor Interfaces"
- note added: "TODO: Add Pullups"
- note added: "USART Port"
- moved on the sheet: C4, C5, C6, C7, C8, D2, F1, FB1, J1, J2, U2, U3

Commit message: Final changes to Sensor Pack
Parts:
- added H1: M3 Bolt, MountingHole:MountingHole_3.2mm_M3, symbol Mechanical:MountingHole
- added TP1, TP2: 1p, Connector_PinHeader_2.54mm:PinHeader_1x01_P2.54mm_Vertical, symbol Connector:TestPoint
- F1: value 200mA Polyfuse -> 1A Polyfuse; Digikey Part (none) -> MF-NSMF050-2
- J1: value M12x5 A-Type -> M12x5 A-Type Female; footprint Capstone_Footprints:M12x5_A_Circular_Connector -> Capstone_Footprints:M12A05PFFRSF7003
- J10: footprint Capstone_Footprints:2x03_2.54mm_DIP_pogo -> Connector_PinHeader_2.54mm:PinHeader_2x03_P2.54mm_Vertical; symbol Capstone_Symbols:Conn_02x03_Counter_Clockwise -> Connector_Generic:Conn_02x03_Odd_Even
- J2: value M12x5 A-Type -> M12x5 A-Type Male; footprint Capstone_Footprints:M12x5_A_Circular_Connector -> Capstone_Footprints:M12A05PMMRSF7003
- JP1, JP2, JP3, JP4, JP5, JP6: Digikey Part (none) -> RMCF0603ZT0R00
- R1: value 4.7k -> 4k7; Digikey Part (none) -> RMCF0603FT4K70
- R10, R14: Digikey Part (none) -> RMCF0603FT1K00
- R11, R15: Digikey Part (none) -> RMCF0603FT2K00
- R12, R13, R16, R17, R8, R9: Digikey Part (none) -> RMCF0603FT4K70
- R2: Digikey Part (none) -> RMCF0603FT2K20
- R3: Digikey Part (none) -> RMCF0603JT47K0
- R6, R7: Digikey Part (none) -> RMCF0603FT10K0
Connections:
- net +3V3: now also J10.4 (Pin_4), TP2.1; no longer J10.5 (Pin_5)
- net +5V: now also TP1.1
- net GND: now also J10.5 (Pin_5), J10.6 (Pin_6); no longer J10.3 (Pin_3), J10.4 (Pin_4)
- net NRST: now also J10.3 (Pin_3); no longer J10.2 (Pin_2)
- net SWCLK: now also J10.2 (Pin_2); no longer J10.6 (Pin_6)
Other:
- note removed: "TODO: Add Pullups"
- company: (none) -> Vector Drive
- title: (none) -> Sensor Pack Board
- moved on the sheet: C6, C7, U3

Commit message: BOM changes, minor schematic change
Parts:
- removed LED1: RG LED, LED_THT:LED_D3.0mm-3, symbol Capstone_Symbols:LED_Dual_KAK
- removed Q1: DMN2310U, Package_TO_SOT_SMD:SOT-23-3, symbol Capstone_Symbols:Q_NMOS_GSD
- added LED1: RG LED, LED_THT:LED_D3.0mm-3, symbol Device:LED_Dual_AKA
- added Q2: TLV75533, Package_DIP:DIP-24_W7.62mm, symbol Transistor_FET:Q_PMOS_DGS
- J10: Digikey Part 1528-5382-ND -> (none)
- R1: value 4k7 -> 330R
- R2: value 2.2k -> 1k
- U2: Digikey Part (none) -> TLV75533PDBVR
- U3: Digikey Part (none) -> STM32C092KCT6
- Y1: value 8MHz 16pF Load -> 8MHz 18pF Load
Connections:
- net +3V3: now also Q2.3 (S); no longer R3.1
- net EN_LED_R: now also R3.1, Q2.2 (G); no longer R3.2
- net GND: now also R3.2, LED1.2 (K)
- net at R2.2: now also LED1.1 (A1)
- net at R1.2: now also LED1.3 (A2)
- net at R2.1: now also Q2.1 (D)

Commit message: Tweaks
Parts:
- C4, C6: Digikey Part CL21A106KOQNNNE -> CL21A106KPCLQNC
- C5, C7, C8: Digikey Part CL10B104KB8NFNC -> CL10B104KO8NNNC
- H1: KiLib_Generator (none) -> mounting_hardware/mounting_hole
- J10, TP1, TP2: KiLib_Generator (none) -> connector/pin_header_socket
- LED1: Digikey Part 5218738F -> WP59SURKZGW
- Q2: value TLV75533 -> DMP2045U-7; footprint Package_DIP:DIP-24_W7.62mm -> Capstone_Footprints:SOT-23-3; symbol Transistor_FET:Q_PMOS_DGS -> Transistor_FET:Q_PMOS_GSD; Digikey Part TLV75533PDBVR -> DMP2045U-7; KiLib_Generator (none) -> package/gullwing
- renumbered R2 to R1, R1 to R2
Connections:
- net +3V3: now also Q2.2 (S); no longer Q2.3 (S)
- net EN_LED_R: now also Q2.1 (G); no longer Q2.2 (G)
- net at R1.1: now also Q2.3 (D); no longer Q2.1 (D)
Changed lines of the file:
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@@
 		(in_pos_files yes)
 		(dnp no)
-		(property "Reference" "R2"
+		(property "Reference" "R1"
 			(at 142.24 175.26 90)
 			(show_name no)
@@
 			(project "SensorPack_v1"
 				(path "/7f033487-c793-47e5-80dd-4bcaea87e7a6"
-					(reference "R2")
+					(reference "R1")
 					(unit 1)
 				)
@@
 			)
 		)
+		(property "KiLib_Generator" "connector/pin_header_socket"
+			(at 73.66 25.4 0)
+			(hide yes)
+			(show_name no)
+			(do_not_autoplace no)
+			(effects
+				(font
+					(size 1.27 1.27)
+				)
+			)
+		)
 		(pin "1"
 		)
@@
 			)
 		)
-		(property "Digikey Part" "CL10B104KB8NFNC"
+		(property "Digikey Part" "CL10B104KO8NNNC"
 			(at 105.41 82.55 0)
 			(hide yes)
@@
 			)
 		)
+		(property "KiLib_Generator" "connector/pin_header_socket"
+			(at 73.66 171.45 0)
+			(hide yes)
+			(show_name no)
+			(do_not_autoplace no)
+			(effects
+				(font
+					(size 1.27 1.27)
+				)
+			)
+		)
 		(pin "3"
 		)
@@
 			)
 		)
-		(property "Digikey Part" "CL21A106KOQNNNE"
+		(property "Digikey Part" "CL21A106KPCLQNC"
 			(at 115.57 82.55 0)
 			(hide yes)
@@
 			)
 		)
-		(property "Digikey Part" "CL21A106KOQNNNE"
+		(property "Digikey Part" "CL21A106KPCLQNC"
 			(at 55.88 34.29 0)
 			(hide yes)
@@
 		(dnp no)
 		(fields_autoplaced yes)
-		(property "Reference" "R1"
+		(property "Reference" "R2"
 			(at 142.24 160.02 90)
 			(show_name no)
@@
 			(project "SensorPack_v1"
 				(path "/7f033487-c793-47e5-80dd-4bcaea87e7a6"
-					(reference "R1")
+					(reference "R2")
 					(unit 1)
 				)
@@
 			)
 		)
-		(property "Digikey Part" "5218738F"
+		(property "Digikey Part" "WP59SURKZGW"
 			(at 153.67 168.91 0)
 			(hide yes)
@@
 			)
 		)
+		(property "KiLib_Generator" "connector/pin_header_socket"
+			(at 113.03 25.4 0)
+			(hide yes)
+			(show_name no)
+			(do_not_autoplace no)
+			(effects
+				(font
+					(size 1.27 1.27)
+				)
+			)
+		)
 		(pin "1"
 		)
@@
 	)
 	(symbol
-		(lib_id "Transistor_FET:Q_PMOS_DGS")
+		(lib_id "Transistor_FET:Q_PMOS_GSD")
 		(at 120.65 172.72 0)
 		(mirror x)
@@
 			)
 		)
-		(property "Value" "TLV75533"
+		(property "Value" "DMP2045U-7"
 			(at 127 171.4501 0)
 			(show_name no)
@@
 			)
 		)
-		(property "Footprint" "Package_DIP:DIP-24_W7.62mm"
+		(property "Footprint" "Capstone_Footprints:SOT-23-3"
 			(at 125.73 175.26 0)
 			(hide yes)
@@
 			)
 		)
-		(property "Description" "P-MOSFET transistor, drain/gate/source"
+		(property "Description" "P-MOSFET transistor, gate/source/drain"
 			(at 120.65 172.72 0)
 			(hide yes)
@@
 			)
 		)
-		(property "Digikey Part" "TLV75533PDBVR"
+		(property "Digikey Part" "DMP2045U-7"
+			(at 120.65 172.72 0)
+			(hide yes)
+			(show_name no)
+			(do_not_autoplace no)
+			(effects
+				(font
+					(size 1.27 1.27)
+				)
+			)
+		)
+		(property "KiLib_Generator" "package/gullwing"
 			(at 120.65 172.72 0)
 			(hide yes)
@@
 			)
 		)
-		(property "Digikey Part" "CL10B104KB8NFNC"
+		(property "Digikey Part" "CL10B104KO8NNNC"
 			(at 105.41 34.29 0)
 			(hide yes)
@@
 			)
 		)
-		(property "Digikey Part" "CL10B104KB8NFNC"
+		(property "Digikey Part" "CL10B104KO8NNNC"
 			(at 64.77 34.29 0)
 			(hide yes)
@@
 			(at 66.04 99.06 0)
 			(hide yes)
+			(show_name no)
+			(do_not_autoplace no)
+			(effects
+				(font
+					(size 1.27 1.27)
+				)
+			)
+		)
+		(property "KiLib_Generator" "mounting_hardware/mounting_hole"
+			(at 66.04 99.06 0)
+			(hide yes)

Commit message: Added some mechanical notes, adjusted traces to not run under bolt (just in case), scooted top connector back in place
Parts:
- J1: Digikey Part (none) -> M12A05PFFRSF7003
- J2: Digikey Part (none) -> M12A05PMMRSF7003
Changed lines of the file:
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@@
 			)
 		)
-		(property "Digikey Part" ""
+		(property "Digikey Part" "M12A05PMMRSF7003"
 			(at 31.75 62.23 0)
 			(hide yes)
@@
 			)
 		)
-		(property "Digikey Part" ""
-			(at 82.55 62.23 0)
-			(hide yes)
+		(property "Digikey Part" "M12A05PFFRSF7003"
+			(at 82.55 62.23 0)
+			(hide yes)
