File: SensorCore_v1/CAN_Transceiver.kicad_sch (KiCad schematic)
At the start: 6 parts, among them U2 MCP2562-E-SN

Commit message: Featured out SensorPack_v1
Other:
- company: (none) -> Vector Drive (MXET)
- title: (none) -> Sensor Core PCB
Changed lines of the file:
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@@
 	(generator_version "10.0")
 	(paper "A4")
+	(title_block
+		(title "Sensor Core PCB")
+		(date "2026-09-08")
+		(rev "v1.1")
+		(company "Vector Drive (MXET)")
+		(comment 1 "Lucas Ngo")
+		(comment 2 "Abhi Chennuru")
+		(comment 3 "Jaden Solorzano")
+		(comment 4 "Rudra Premani")
+		(comment 5 "Yi-Cheng Quan")
+	)
 	(junction
 		(at 49.53 69.85)

Commit message: Preliminary design done
Parts:
- C3: renamed from C8; footprint Resistor_SMD:R_0603_1608Metric_Pad0.98x0.95mm_HandSolder -> Capstone Footprints:C_0603_1608Metric_Pad1.08x0.95mm_HandSolder; symbol Device:C -> Project:C; KiLib_Generator (none) -> SMD_2terminal_chip_molded
- CM1: footprint Extra_Footprints:CMChoke_2.6x1.2mm_HandSolder -> Capstone Footprints:CMChoke_2.6x1.2mm_HandSolder; symbol Device:L_Ferrite_Coupled -> Project:L_Ferrite_Coupled
- D1: footprint Package_TO_SOT_SMD:SOT-23-3 -> Capstone Footprints:SOT-23-3; symbol Device:D_TVS_Dual_AAC -> Project:D_TVS_Dual_AAC
- R1: renamed from R2; footprint Resistor_SMD:R_0603_1608Metric_Pad0.98x0.95mm_HandSolder -> Capstone Footprints:R_0603_1608Metric_Pad0.98x0.95mm_HandSolder; symbol Device:R -> Project:R
- R2: renamed from R3; footprint Resistor_SMD:R_0603_1608Metric_Pad0.98x0.95mm_HandSolder -> Capstone Footprints:R_0603_1608Metric_Pad0.98x0.95mm_HandSolder; symbol Device:R -> Project:R
- U1: renamed from U2; footprint Package_SO:SOIC-8_3.9x4.9mm_P1.27mm -> Capstone Footprints:SOIC-8_3.9x4.9mm_P1.27mm; symbol Interface_CAN_LIN:MCP2562-E-SN -> Project:MCP2562-E-SN; KiLib_Generator (none) -> package/gullwing
Connections:
- net Net-(U2-CANL): now reaches CM1.2, U1.6 (CANL)
- net Net-(U2-CANH): now reaches CM1.4, U1.7 (CANH)
Changed lines of the file:
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@@
+		)
+	)
+	(label "Net-(U2-CANH)"
+		(at 81.28 69.85 180)
+		(effects
+			(font
+				(size 1.27 1.27)
+			)
+			(justify right bottom)
+		)
+	)
+	(label "Net-(U2-CANL)"
+		(at 81.28 74.93 180)
+		(effects
+			(font
+				(size 1.27 1.27)
+			)
+			(justify right bottom)
+		)
+	)
+	(label "Net-(U2-CANH)"
+		(at 81.28 69.85 180)
+		(effects
+			(font
+				(size 1.27 1.27)
+			)
+			(justify right bottom)
+		)
+	)
+	(label "Net-(U2-CANL)"
+		(at 81.28 74.93 180)
+		(effects
+			(font
+				(size 1.27 1.27)
+			)
+			(justify right bottom)
 		)
 	)
@@
 	)
 	(symbol
-		(lib_id "Device:R")
+		(lib_id "Project:R")
 		(at 44.45 74.93 270)
 		(mirror x)
@@
 		(dnp no)
 		(fields_autoplaced yes)
-		(property "Reference" "R3"
+		(property "Reference" "R2"
 			(at 44.45 78.74 90)
 			(show_name no)
@@
 			)
 		)
-		(property "Footprint" "Resistor_SMD:R_0603_1608Metric_Pad0.98x0.95mm_HandSolder"
+		(property "Footprint" "Capstone Footprints:R_0603_1608Metric_Pad0.98x0.95mm_HandSolder"
 			(at 44.45 76.708 90)
 			(hide yes)
@@
 		)
 		(property "Digikey Part" ""
+			(at 44.45 74.93 90)
+			(hide yes)
+			(show_name no)
+			(do_not_autoplace no)
+			(effects
+				(font
+					(size 1.27 1.27)
+				)
+			)
+		)
+		(property "Sim.Device" ""
+			(at 44.45 74.93 90)
+			(hide yes)
+			(show_name no)
+			(do_not_autoplace no)
+			(effects
+				(font
+					(size 1.27 1.27)
+				)
+			)
+		)
+		(property "Sim.Pins" ""
 			(at 44.45 74.93 90)
 			(hide yes)
@@
 			(project "SensorCore_v1"
 				(path "/7f033487-c793-47e5-80dd-4bcaea87e7a6/48e3238f-f116-44df-bab8-01919a7a82f8"
-					(reference "R3")
+					(reference "R2")
 					(unit 1)
 				)
@@
 	)
 	(symbol
-		(lib_id "Interface_CAN_LIN:MCP2562-E-SN")
+		(lib_id "Project:MCP2562-E-SN")
 		(at 93.98 72.39 0)
 		(mirror y)
@@
 		(dnp no)
 		(fields_autoplaced yes)
-		(property "Reference" "U2"
+		(property "Reference" "U1"
 			(at 97.0981 59.69 0)
 			(show_name no)
@@
 			)
 		)
-		(property "Footprint" "Package_SO:SOIC-8_3.9x4.9mm_P1.27mm"
+		(property "Footprint" "Capstone Footprints:SOIC-8_3.9x4.9mm_P1.27mm"
 			(at 93.98 85.09 0)
 			(hide yes)
@@
 		)
 		(property "Description" "High-Speed CAN Transceiver, 1Mbps, 5V supply, Vio pin, -40C to +125C, SOIC-8"
+			(at 93.98 72.39 0)
+			(hide yes)
+			(show_name no)
+			(do_not_autoplace no)
+			(effects
+				(font
+					(size 1.27 1.27)
+				)
+			)
+		)
+		(property "Sim.Device" ""
+			(at 93.98 72.39 0)
+			(hide yes)
+			(show_name no)
+			(do_not_autoplace no)
+			(effects
+				(font
+					(size 1.27 1.27)
+				)
+			)
+		)
+		(property "Sim.Pins" ""
+			(at 93.98 72.39 0)
+			(hide yes)
+			(show_name no)
+			(do_not_autoplace no)
+			(effects
+				(font
+					(size 1.27 1.27)
+				)
+			)
+		)
+		(property "KiLib_Generator" "package/gullwing"
 			(at 93.98 72.39 0)
 			(hide yes)
@@
 			(project "SensorCore_v1"
 				(path "/7f033487-c793-47e5-80dd-4bcaea87e7a6/48e3238f-f116-44df-bab8-01919a7a82f8"
-					(reference "U2")
+					(reference "U1")
 					(unit 1)
 				)
@@
 	)
 	(symbol
-		(lib_id "Device:C")
+		(lib_id "Project:C")
 		(at 88.9 53.34 0)
 		(mirror y)
@@
 		(dnp no)
 		(fields_autoplaced yes)
-		(property "Reference" "C8"
+		(property "Reference" "C3"
 			(at 85.09 52.0699 0)
 			(show_name no)
@@
 			)
 		)
-		(property "Footprint" "Resistor_SMD:R_0603_1608Metric_Pad0.98x0.95mm_HandSolder"
+		(property "Footprint" "Capstone Footprints:C_0603_1608Metric_Pad1.08x0.95mm_HandSolder"
 			(at 87.9348 57.15 0)
 			(hide yes)
@@
 		)
 		(property "Digikey Part" "CL10B104KB8NFNC"
+			(at 88.9 53.34 0)
+			(hide yes)
+			(show_name no)
+			(do_not_autoplace no)
+			(effects
+				(font
+					(size 1.27 1.27)
+				)
+			)
+		)
+		(property "Sim.Device" ""
+			(at 88.9 53.34 0)
+			(hide yes)
+			(show_name no)
+			(do_not_autoplace no)
+			(effects
+				(font
+					(size 1.27 1.27)
+				)
+			)
+		)
+		(property "Sim.Pins" ""
+			(at 88.9 53.34 0)
+			(hide yes)
+			(show_name no)
+			(do_not_autoplace no)
+			(effects
+				(font
+					(size 1.27 1.27)
+				)
+			)
+		)
+		(property "KiLib_Generator" "SMD_2terminal_chip_molded"
 			(at 88.9 53.34 0)
 			(hide yes)
@@
 			(project "SensorCore_v1"
 				(path "/7f033487-c793-47e5-80dd-4bcaea87e7a6/48e3238f-f116-44df-bab8-01919a7a82f8"
-					(reference "C8")
+					(reference "C3")
 					(unit 1)
 				)
@@
 	)
 	(symbol
-		(lib_id "Device:D_TVS_Dual_AAC")
+		(lib_id "Project:D_TVS_Dual_AAC")
 		(at 58.42 85.09 0)
 		(unit 1)
@@
 			)
 		)
-		(property "Footprint" "Package_TO_SOT_SMD:SOT-23-3"
+		(property "Footprint" "Capstone Footprints:SOT-23-3"
 			(at 54.61 85.09 0)
 			(hide yes)
@@
 		)
 		(property "Digikey Part" "DESD12VL2BTQ-7"
+			(at 58.42 85.09 0)
+			(hide yes)
+			(show_name no)
+			(do_not_autoplace no)
+			(effects
+				(font
+					(size 1.27 1.27)
+				)
+			)
+		)
+		(property "Sim.Device" ""
+			(at 58.42 85.09 0)
+			(hide yes)
+			(show_name no)
+			(do_not_autoplace no)
+			(effects
+				(font
+					(size 1.27 1.27)
+				)
+			)
+		)
+		(property "Sim.Pins" ""
 			(at 58.42 85.09 0)
 			(hide yes)
@@
 	)
 	(symbol
-		(lib_id "Device:R")
+		(lib_id "Project:R")
 		(at 44.45 69.85 270)
 		(mirror x)
@@
 		(dnp no)
 		(fields_autoplaced yes)
-		(property "Reference" "R2"
+		(property "Reference" "R1"
 			(at 44.45 63.5 90)
 			(show_name no)
@@
 			)
 		)
-		(property "Footprint" "Resistor_SMD:R_0603_1608Metric_Pad0.98x0.95mm_HandSolder"
+		(property "Footprint" "Capstone Footprints:R_0603_1608Metric_Pad0.98x0.95mm_HandSolder"
 			(at 44.45 71.628 90)
 			(hide yes)
@@
 		)
 		(property "Digikey Part" ""
+			(at 44.45 69.85 90)
+			(hide yes)
+			(show_name no)
+			(do_not_autoplace no)
+			(effects
+				(font
+					(size 1.27 1.27)
+				)
+			)
+		)
+		(property "Sim.Device" ""
+			(at 44.45 69.85 90)
+			(hide yes)
+			(show_name no)
+			(do_not_autoplace no)
+			(effects
+				(font
+					(size 1.27 1.27)
+				)
+			)
+		)
+		(property "Sim.Pins" ""
 			(at 44.45 69.85 90)
 			(hide yes)
@@
 			(project "SensorCore_v1"
 				(path "/7f033487-c793-47e5-80dd-4bcaea87e7a6/48e3238f-f116-44df-bab8-01919a7a82f8"
-					(reference "R2")
+					(reference "R1")
 					(unit 1)
 				)
@@
 	)
 	(symbol
-		(lib_id "Device:L_Ferrite_Coupled")
+		(lib_id "Project:L_Ferrite_Coupled")
 		(at 73.66 72.39 0)
 		(mirror x)
@@
 			)
 		)
-		(property "Footprint" "Extra_Footprints:CMChoke_2.6x1.2mm_HandSolder"
+		(property "Footprint" "Capstone Footprints:CMChoke_2.6x1.2mm_HandSolder"
 			(at 73.66 72.39 0)
 			(hide yes)
@@
 			(at 73.66 72.39 0)
 			(hide yes)
+			(show_name no)
+			(do_not_autoplace no)
+			(effects
+				(font
+					(size 1.27 1.27)
+				)
+			)
+		)
+		(property "Sim.Device" ""
+			(at 73.66 72.39 0)
+			(hide yes)
+			(show_name no)
+			(do_not_autoplace no)
+			(effects
+				(font
+					(size 1.27 1.27)
+				)
+			)
+		)
+		(property "Sim.Pins" ""
+			(at 73.66 72.39 0)
+			(hide yes)

Commit message: SensorCore v1.0 - Approved
Parts:
- U1: Digikey Part (none) -> MCP2562-E-SN
Connections:
- net CANH: now also D1.1 (A1)
- net CANL: now also D1.2 (A2)
- net at CM1.1, R2.1: no longer D1.2 (A2)
- net at CM1.3, R1.1: no longer D1.1 (A1)
- net Net-(U2-CANH): no longer names the net of CM1.4, U1.7 (CANH)
- net Net-(U2-CANL): no longer names the net of CM1.2, U1.6 (CANL)
Other:
- moved on the sheet: D1
