File: SensorCore_v1/SensorCore_v1.kicad_pcb (KiCad board)
At the start: 4 copper layers, 37 parts, among them J1 Micro_SD_Card_Det1, J2 M12x5 A-Type, J3 2x3 Header, J4 M12x5 A-Type, Q1 DMN2310U, U1 STM32C092KCT6, U2 ATA6563, U3 R-78K3.3-1.0, U4 EMIF06-MSD02N16, Y1 8MHz 16pF Load

Commit message: Preliminary design done
Parts:
- removed the C4 at (97.3, 57.9)
- removed the C5 at (109.0, 75.8)
- removed the C6 at (109.0, 78.8)
- removed the R6 at (101.7, 63.0)
- removed the U3 at (99.2, 67.1)
- added C1: 10uF 16V, Capstone Footprints:C_0805_2012Metric_Pad1.18x1.45mm_HandSolder, F.Cu at (118.1, 104.6)
- added C11: 10uF 16V, Capstone Footprints:C_0805_2012Metric_Pad1.18x1.45mm_HandSolder, F.Cu at (96.0, 134.8)
- added C13: 100nF, Capstone Footprints:C_0603_1608Metric_Pad1.08x0.95mm_HandSolder, F.Cu at (94.2, 134.8)
- added C15: 100nF, Capstone Footprints:C_0603_1608Metric_Pad1.08x0.95mm_HandSolder, F.Cu at (86.0, 141.2)
- added C17: 10uF 50V, Capstone Footprints:C_0805_2012Metric_Pad1.18x1.45mm_HandSolder, F.Cu at (79.0, 143.2)
- added C18: 33u, Capstone Footprints:CP_Radial_D6.3mm_P2.50mm, F.Cu at (74.5, 135.2)
- added C19: 10uF 50V, Capstone Footprints:C_0805_2012Metric_Pad1.18x1.45mm_HandSolder, F.Cu at (71.5, 123.3)
- added C2: 100nF, Capstone Footprints:C_0603_1608Metric_Pad1.08x0.95mm_HandSolder, F.Cu at (116.3, 104.8)
- added C20: 10uF 50V, Capstone Footprints:C_0805_2012Metric_Pad1.18x1.45mm_HandSolder, F.Cu at (71.5, 127.8)
- added C8: 10uF 16V, Capstone Footprints:C_0805_2012Metric_Pad1.18x1.45mm_HandSolder, F.Cu at (98.0, 127.2)
- added C9: 10uF 16V, Capstone Footprints:C_0805_2012Metric_Pad1.18x1.45mm_HandSolder, F.Cu at (98.0, 134.8)
- added D2: 12V TVS 1CH, Capstone Footprints:D_SMA, F.Cu at (97.0, 131.0)
- added D4: 12V Zener, Capstone Footprints:D_SOD-123, F.Cu at (74.2, 148.1)
- added H1: M3 Bolt, Capstone Footprints:MountingHole_3.2mm_M3, F.Cu at (117.5, 130.0)
- added H2: M3 Bolt, Capstone Footprints:MountingHole_3.2mm_M3, F.Cu at (73.5, 103.5)
- added H3: M3 Bolt, Capstone Footprints:MountingHole_3.2mm_M3, F.Cu at (73.5, 156.5)
- added J1: 2x3 Pogo Header, Capstone Footprints:PinHeader_2x03_P2.54mm_Vertical, F.Cu at (122.5, 104.8)
- added J5: 6p JST-XH, Capstone Footprints:JST_XH_B6B-XH-A_1x06_P2.50mm_Vertical, F.Cu at (108.0, 155.8)
- added J6: 4p JST-XH, Capstone Footprints:JST_XH_B4B-XH-A_1x04_P2.50mm_Vertical, F.Cu at (100.0, 155.8)
- added J7: 4p JST-XH, Capstone Footprints:JST_XH_B4B-XH-A_1x04_P2.50mm_Vertical, F.Cu at (92.0, 155.8)
- added J9: 2p JST-XH, Capstone Footprints:JST_XH_B2B-XH-A_1x02_P2.50mm_Vertical, F.Cu at (80.0, 155.8)
- added L1: 5u6, Capstone Footprints:IFSC2020DEER5R6M01, F.Cu at (76.8, 122.1)
- added L2: 5u6, Capstone Footprints:IFSC2020DEER5R6M01, F.Cu at (76.8, 129.3)
- added Q2: DMP2045U-7, Capstone Footprints:SOT-23-3, F.Cu at (74.6, 141.6)
- added Q3: DMP2045U-7, Capstone Footprints:SOT-23-3, F.Cu at (74.6, 145.1)
- added R10: 47k, Capstone Footprints:R_0603_1608Metric_Pad0.98x0.95mm_HandSolder, F.Cu at (98.4, 120.0)
- added R11: 330R, Capstone Footprints:R_0603_1608Metric_Pad0.98x0.95mm_HandSolder, F.Cu at (96.9, 119.8)
- added R12: 4k7, Capstone Footprints:R_0603_1608Metric_Pad0.98x0.95mm_HandSolder, F.Cu at (94.2, 143.0)
- added R13: 4k7, Capstone Footprints:R_0603_1608Metric_Pad0.98x0.95mm_HandSolder, F.Cu at (94.2, 144.5)
- added R14: 4k7, Capstone Footprints:R_0603_1608Metric_Pad0.98x0.95mm_HandSolder, F.Cu at (91.8, 139.5)
- added R15: 4k7, Capstone Footprints:R_0603_1608Metric_Pad0.98x0.95mm_HandSolder, F.Cu at (90.2, 139.5)
- added R16: 100m, Capstone Footprints:R_0805_2012Metric_Pad1.20x1.40mm_HandSolder, F.Cu at (79.0, 139.8)
- added R17: 33k, Capstone Footprints:R_0603_1608Metric_Pad0.98x0.95mm_HandSolder, F.Cu at (74.8, 150.0)
- added R18: 1k, Capstone Footprints:R_0603_1608Metric_Pad0.98x0.95mm_HandSolder, F.Cu at (74.8, 151.5)
- added R3: 4k7, Capstone Footprints:R_0603_1608Metric_Pad0.98x0.95mm_HandSolder, F.Cu at (119.8, 104.8)
- added R4: 4k7, Capstone Footprints:R_0603_1608Metric_Pad0.98x0.95mm_HandSolder, F.Cu at (110.2, 138.0)
- added R8: 4k7, Capstone Footprints:R_0603_1608Metric_Pad0.98x0.95mm_HandSolder, F.Cu at (102.2, 143.0)
- added R9: 4k7, Capstone Footprints:R_0603_1608Metric_Pad0.98x0.95mm_HandSolder, F.Cu at (102.2, 144.5)
- added SW1: SWS065, Capstone Footprints:SW_SWS065-030V12TSK_REVA, F.Cu at (86.5, 153.2)
- added U1: MCP2562-E-SN, Capstone Footprints:SOIC-8_3.9x4.9mm_P1.27mm, F.Cu at (115.0, 152.2)
- added U5: INA226, Capstone Footprints:TSSOP-10_3x3mm_P0.5mm, F.Cu at (86.0, 138.8)
- added U6: R-78C5.0-1.0, Capstone Footprints:Converter_DCDC_RECOM_R-78E-0.5_THT, F.Cu at (84.8, 125.2)
- added U7: R-78C3.3-1.0, Capstone Footprints:Converter_DCDC_RECOM_R-78E-0.5_THT, F.Cu at (84.8, 134.4)
- C10: footprint Capacitor_SMD:C_0805_2012Metric_Pad1.18x1.45mm_HandSolder -> Capstone Footprints:C_0805_2012Metric_Pad1.18x1.45mm_HandSolder
- C12: footprint Resistor_SMD:R_0603_1608Metric_Pad0.98x0.95mm_HandSolder -> Capstone Footprints:C_0603_1608Metric_Pad1.08x0.95mm_HandSolder
- C14: renamed from C3; footprint Resistor_SMD:R_0603_1608Metric_Pad0.98x0.95mm_HandSolder -> Capstone Footprints:C_0603_1608Metric_Pad1.08x0.95mm_HandSolder
- C16: renamed from C11; footprint Capacitor_SMD:C_0805_2012Metric_Pad1.18x1.45mm_HandSolder -> Capstone Footprints:C_0805_2012Metric_Pad1.18x1.45mm_HandSolder
- C3: renamed from C8; footprint Resistor_SMD:R_0603_1608Metric_Pad0.98x0.95mm_HandSolder -> Capstone Footprints:C_0603_1608Metric_Pad1.08x0.95mm_HandSolder
- C4: renamed from C1; footprint Capacitor_SMD:C_0603_1608Metric_Pad1.08x0.95mm_HandSolder -> Capstone Footprints:C_0603_1608Metric_Pad1.08x0.95mm_HandSolder
- C5: renamed from C2; footprint Capacitor_SMD:C_0603_1608Metric_Pad1.08x0.95mm_HandSolder -> Capstone Footprints:C_0603_1608Metric_Pad1.08x0.95mm_HandSolder
- C6: renamed from C7; footprint Resistor_SMD:R_0603_1608Metric_Pad0.98x0.95mm_HandSolder -> Capstone Footprints:C_0603_1608Metric_Pad1.08x0.95mm_HandSolder
- C7: renamed from C9; footprint Capacitor_SMD:C_0805_2012Metric_Pad1.18x1.45mm_HandSolder -> Capstone Footprints:C_0805_2012Metric_Pad1.18x1.45mm_HandSolder
- CM1: footprint Extra_Footprints:CMChoke_2.6x1.2mm_HandSolder -> Capstone Footprints:CMChoke_2.6x1.2mm_HandSolder
- D1: footprint Package_TO_SOT_SMD:SOT-23-3 -> Capstone Footprints:SOT-23-3
- D3: footprint Diode_SMD:D_SMA -> Capstone Footprints:D_SMA
- F1: value 100mA Polyfuse -> 1A Polyfuse; footprint Resistor_SMD:R_1206_3216Metric_Pad1.30x1.75mm_HandSolder -> Capstone Footprints:R_1206_3216Metric_Pad1.30x1.75mm_HandSolder
- FB1: footprint Resistor_SMD:R_0603_1608Metric_Pad0.98x0.95mm_HandSolder -> Capstone Footprints:R_0603_1608Metric_Pad0.98x0.95mm_HandSolder
- J10: renamed from TH1; footprint Resistor_SMD:R_0603_1608Metric_Pad0.98x0.95mm_HandSolder -> Capstone Footprints:JST_XH_B2B-XH-A_1x02_P2.50mm_Vertical
- J2: value M12x5 A-Type -> M12x5 A-Type Female; footprint Extra_Footprints:M12x5_A_Circular_Connector -> Capstone Footprints:M12A05PFFRSF7003
- J3: value 2x3 Header -> M12x5 A-Type Female; footprint Extra_Footprints:2x03_2.54mm_DIP_pogo -> Capstone Footprints:M12A05PFFRSF7003
- J4: value M12x5 A-Type -> 2x3 Pogo Header; footprint Extra_Footprints:M12x5_A_Circular_Connector -> Capstone Footprints:PinHeader_2x03_P2.54mm_Vertical
- J8: renamed from J1; footprint Extra_Footprints:CUI_MSD-11-A -> Capstone Footprints:CUI_MSD-11-A
- LED1: footprint Connector_PinHeader_2.54mm:PinHeader_1x03_P2.54mm_Vertical -> Capstone Footprints:LED_D3.0mm-3
- Q1: value DMN2310U -> DMP2045U-7; footprint Package_TO_SOT_SMD:SOT-23-3 -> Capstone Footprints:SOT-23-3
- R1: renamed from R2; footprint Resistor_SMD:R_0603_1608Metric_Pad0.98x0.95mm_HandSolder -> Capstone Footprints:R_0603_1608Metric_Pad0.98x0.95mm_HandSolder
- R19: renamed from R4; footprint Resistor_SMD:R_0603_1608Metric_Pad0.98x0.95mm_HandSolder -> Capstone Footprints:R_0603_1608Metric_Pad0.98x0.95mm_HandSolder
- R2: renamed from R3; footprint Resistor_SMD:R_0603_1608Metric_Pad0.98x0.95mm_HandSolder -> Capstone Footprints:R_0603_1608Metric_Pad0.98x0.95mm_HandSolder
- R5: value 1k -> 4k7; footprint Resistor_SMD:R_0603_1608Metric_Pad0.98x0.95mm_HandSolder -> Capstone Footprints:R_0603_1608Metric_Pad0.98x0.95mm_HandSolder
- R6: renamed from R1; footprint Resistor_SMD:R_0603_1608Metric_Pad0.98x0.95mm_HandSolder -> Capstone Footprints:R_0603_1608Metric_Pad0.98x0.95mm_HandSolder
- R7: value 47k -> 1k; footprint Resistor_SMD:R_0603_1608Metric_Pad0.98x0.95mm_HandSolder -> Capstone Footprints:R_0603_1608Metric_Pad0.98x0.95mm_HandSolder
- TH1: renamed from TH2; footprint Resistor_SMD:R_0603_1608Metric_Pad0.98x0.95mm_HandSolder -> Capstone Footprints:R_0603_1608Metric_Pad0.98x0.95mm_HandSolder
- U2: value ATA6563 -> RAK3172-9-SM-I; footprint Package_SO:SOIC-8_3.9x4.9mm_P1.27mm -> Capstone Footprints:RAK3172
- U3: renamed from U1; footprint Package_QFP:LQFP-32_7x7mm_P0.8mm -> Capstone Footprints:LQFP-32_7x7mm_P0.8mm
- U4: footprint Package_DFN_QFN:OnSemi_UDFN-16-1EP_1.35x3.3mm_P0.4mm_EP0.4x2.8mm -> Capstone Footprints:OnSemi_UDFN-16-1EP_1.35x3.3mm_P0.4mm_EP0.4x2.8mm
- Y1: footprint Extra_Footprints:Crystal_6x3.5mm -> Capstone Footprints:Crystal_6x3.5mm
- moved D3 91.9 mm to (80.5, 146.0)
- moved FB1 91.5 mm to (79.0, 141.5)
- moved F1 84.7 mm to (79.5, 149.0)
- moved R5 79.5 mm to (110.2, 139.5)
- moved C16 78.7 mm to (85.5, 115.7), turned to -90 degrees
- moved C14 75.2 mm to (87.3, 115.5), turned to 90 degrees
- moved J4 72.7 mm to (113.7, 139.5)
- moved C5 70.6 mm to (112.3, 124.4), turned to 90 degrees
- moved U4 70.6 mm to (90.0, 115.6), turned to 90 degrees
- moved C4 69.6 mm to (112.3, 120.9), turned to -90 degrees
- moved J3 68.8 mm to (120.7, 140.7), turned to 90 degrees
- moved Y1 68.1 mm to (115.5, 122.6), turned to -90 degrees
- moved R7 67.1 mm to (103.4, 120.0), turned to -90 degrees
- moved R6 66.8 mm to (107.1, 122.0), turned to 90 degrees
- moved J10 66.1 mm to (76.2, 114.5)
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Connections:
- net /OSC+ renamed /HS_OSC+
- net /OSC- renamed /HS_OSC-
- CM1 pad 1: Net-(CM1-Pad1) -> Net-(D1-A2)
- CM1 pad 3: Net-(CM1-Pad3) -> Net-(D1-A1)
- D1 pad 1: /CANH -> Net-(D1-A1)
- D1 pad 2: /CANL -> Net-(D1-A2)
- F1 pad 2: +5Vin -> VBat_in
- FB1 pad 1: Net-(D3-A1) -> Net-(Q3-D)
- FB1 pad 2: +5V -> Net-(U6-Vbus)
- J2 pad 1: +5Vin -> +5V
- J2 pad 5: unconnected-(J2-Pin_5-Pad5) -> /ALERT
- J3 pad 1: /SWDIO -> +5V
- J3 pad 2: /NRST -> /CANH
- J3 pad 4: GND -> /CANL
- J3 pad 5: +3V3 -> /ALERT
- J4 pad 1: +5Vin -> /SWDIO
- J4 pad 2: /CANH -> /SWCLK
- J4 pad 3: GND -> /NRST
- J4 pad 4: /CANL -> +3V3
- J4 pad 5: unconnected-(J4-Pin_5-Pad5) -> GND
- J8 pad 9: /SD_Card/Card Detect -> /CARD_DETECT
- LED1 pad 1: Net-(LED1-K1) -> Net-(LED1-A1)
- LED1 pad 2: +5V -> GND
- LED1 pad 3: Net-(LED1-K2) -> Net-(LED1-A2)
- Q1 pad 2: GND -> +3V3
- Q1 pad 3: Net-(Q1-D) -> Net-(Q2-D)
- R1 pad 1: Net-(CM1-Pad3) -> Net-(D1-A1)
- R2 pad 1: Net-(CM1-Pad1) -> Net-(D1-A2)
- R5 pad 1: /EN_LED_G -> +3V3
- R5 pad 2: Net-(LED1-K2) -> /I2C1_SCL2
- R7 pad 1: +3V3 -> Net-(Q2-D)
- R7 pad 2: /EN_LED_R -> Net-(LED1-A1)
- U2 pad 1: /CAN_TXD -> unconnected-(U7-UART2_RX/PA3-Pad1)
- U2 pad 2: GND -> unconnected-(U7-UART2_TX/PA2-Pad2)
- U2 pad 3: +5V -> unconnected-(U7-PA15/PIN_A4-Pad3)
- U2 pad 4: /CAN_RXD -> /USART2_TX
- U2 pad 5: +3V3 -> /USART2_RX
- U2 pad 6: Net-(U2-CANL) -> unconnected-(U7-PA1-Pad6)
- U2 pad 7: Net-(U2-CANH) -> /Wireless Module/RAK3172_SWDIO
- U2 pad 8: /TRANSCEIVER_STBY -> /Wireless Module/RAK3172_SWCLK
- U3 pad 1: /EN_LED_G -> /CAN_TXD
- U3 pad 10: unconnected-(U1-PA3-Pad10) -> /USART2_TX
- U3 pad 11: unconnected-(U1-PA4-Pad11) -> /SPI1_CS1
- U3 pad 12: unconnected-(U1-PA5-Pad12) -> /SPI1_SCK
- U3 pad 13: unconnected-(U1-PA6-Pad13) -> /SPI1_MISO
- U3 pad 14: unconnected-(U1-PA7-Pad14) -> /SPI1_MOSI
- U3 pad 15: unconnected-(U1-PB0-Pad15) -> /EN_LED_R
- U3 pad 16: unconnected-(U1-PB1-Pad16) -> /EN_LED_G
- U3 pad 17: unconnected-(U1-PB2-Pad17) -> /CARD_DETECT
- U3 pad 19: unconnected-(U1-PA9-Pad19) -> /I2C1_SCL1
- U3 pad 20: unconnected-(U1-PC6-Pad20) -> /GNSS_TIMPULSE
- U3 pad 21: unconnected-(U1-PA10-Pad21) -> /I2C1_SDA1
- U3 pad 22: unconnected-(U1-PA11[PA9]-Pad22) -> /I2C2_SCL1
- U3 pad 23: unconnected-(U1-PA12[PA10]-Pad23) -> /I2C2_SDA1
- U3 pad 26: unconnected-(U1-PA15-Pad26) -> /GNSS_RESET
- U3 pad 27: unconnected-(U1-PB3-Pad27) -> /I2C2_SCL2
- U3 pad 28: unconnected-(U1-PB4-Pad28) -> /I2C2_SDA2
- U3 pad 29: /CAN_RXD -> /TRANSCEIVER_STBY
- U3 pad 30: /CAN_TXD -> /I2C1_SCL2
- U3 pad 31: /TRANSCEIVER_STBY -> /I2C1_SDA2
- U3 pad 32: /EN_LED_R -> /CAN_RXD
- U3 pad 9: unconnected-(U1-PA2-Pad9) -> /USART2_RX
- U4 pad 1: /SD_Card/Card Detect -> /CARD_DETECT
- U4 pad 4: /SD_Card/CS -> /SPI1_CS1
- U4 pad 5: /SD_Card/DI -> /SPI1_MOSI
- U4 pad 6: /SD_Card/SCLK -> /SPI1_SCK
- U4 pad 7: /SD_Card/DO -> /SPI1_MISO
Routing:
- net +5V: track 0.00 -> 93.2 mm, vias 0 -> 1
- net /CANH: track 0.00 -> 52.2 mm
- net /CANL: track 0.00 -> 46.7 mm
- net /VNTC2: track 0.00 -> 40.8 mm, vias 0 -> 1
- net Net-(LED1-A1): track 0.00 -> 34.7 mm, vias 0 -> 1
- net +3V3: track 9.52 -> 44.2 mm, vias 3 -> 18
- net VBat: track 0.00 -> 32.5 mm
- net /CARD_DETECT: track 0.00 -> 32.4 mm, vias 0 -> 4
- net /ALERT: track 0.00 -> 28.5 mm
- net /TRANSCEIVER_STBY: track 0.00 -> 27.9 mm, vias 0 -> 2
- net /Wireless Module/RAK3172_SWCLK: track 0.00 -> 27.7 mm, vias 0 -> 1
- net /Wireless Module/RAK3172_SWDIO: track 0.00 -> 26.6 mm, vias 0 -> 1
- net /NRST: track 0.00 -> 25.6 mm, vias 0 -> 1
- net Net-(LED1-A2): track 0.00 -> 24.9 mm, vias 0 -> 1
- net /CAN_RXD: track 0.00 -> 24.6 mm
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- added copper zone on In2.Cu, net +3V3
- added copper zone on B.Cu, net GND
- added copper zone on F.Cu, net GND
- added copper zone on In1.Cu, net GND
Other:
- board outline added: 60 x 60 mm

Commit message: SensorCore v1.0 - Approved
Parts:
- added C21: 1n, Capstone Footprints:C_0603_1608Metric_Pad1.08x0.95mm_HandSolder, F.Cu at (87.0, 139.0)
- added C22: 1n, Capstone Footprints:C_0603_1608Metric_Pad1.08x0.95mm_HandSolder, F.Cu at (87.2, 128.2)
- added R20: 1k, Capstone Footprints:R_0603_1608Metric_Pad0.98x0.95mm_HandSolder, F.Cu at (79.0, 143.5)
- added R21: 0R, Capstone Footprints:R_0603_1608Metric_Pad0.98x0.95mm_HandSolder, F.Cu at (97.0, 115.9)
- added R22: 0R, Capstone Footprints:R_0603_1608Metric_Pad0.98x0.95mm_HandSolder, F.Cu at (95.2, 115.9)
- L1, L2: value 5u6 -> 18u
- U6: value R-78C5.0-1.0 -> R-78K5.0-1.0
- U7: value R-78C3.3-1.0 -> R-78K3.3-1.0
- moved D2 25.9 mm to (117.1, 114.6), turned to 90 degrees
- moved U5 5.03 mm to (88.2, 143.2)
- moved R1 4.82 mm to (122.2, 156.5)
- moved R2 4.82 mm to (122.2, 158.0)
- moved R15 4.47 mm to (94.2, 141.5), turned to 180 degrees
- moved D1 3.25 mm to (126.0, 155.8)
- moved R16 2.58 mm to (79.8, 137.3), turned to 90 degrees
- moved R14 2.55 mm to (94.2, 140.0), turned to 180 degrees
- moved U7 1.51 mm to (84.8, 136.0)
- moved C17 1.50 mm to (79.0, 141.8), turned to 0 degrees
- moved FB1 1.50 mm to (79.0, 140.0)
- moved C15 1.25 mm to (87.0, 140.5)
- moved D3 0.90 mm to (81.4, 146.0)
- moved F1 0.90 mm to (80.4, 149.0)
- moved C18 0.56 mm to (75.0, 135.0)
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Connections:
- CM1 pad 1: Net-(D1-A2) -> Net-(CM1-Pad1)
- CM1 pad 3: Net-(D1-A1) -> Net-(CM1-Pad3)
- D1 pad 1: Net-(D1-A1) -> /CANH
- D1 pad 2: Net-(D1-A2) -> /CANL
- D4 pad 2: Net-(D2-A) -> Net-(D4-A)
- Q2 pad 1: Net-(D2-A) -> Net-(D4-A)
- Q3 pad 1: Net-(D2-A) -> Net-(Q3-G)
- R1 pad 1: Net-(D1-A1) -> Net-(CM1-Pad3)
- R17 pad 1: Net-(D2-A) -> Net-(D4-A)
- R18 pad 2: Net-(D2-A) -> Net-(D4-A)
- R2 pad 1: Net-(D1-A2) -> Net-(CM1-Pad1)
- U2 pad 4: /USART2_TX -> /Wireless Module/RAK3172_TX
- U2 pad 5: /USART2_RX -> /Wireless Module/RAK3172_RX
- U3 pad 10: /USART2_TX -> /USART2_RX
- U3 pad 9: /USART2_RX -> /USART2_TX
Routing:
- net Net-(D2-A): track 13.6 -> 0.00 mm
- net Net-(D4-A): track 0.00 -> 13.5 mm, vias 0 -> 2
- net /Wireless Module/RAK3172_RX: track 0.00 -> 11.2 mm
- net /Wireless Module/RAK3172_TX: track 0.00 -> 10.3 mm
- net Net-(D1-A1): track 9.87 -> 0.00 mm
- net Net-(D1-A2): track 9.13 -> 0.00 mm
- net /CANH: track 52.2 -> 60.2 mm
- net /CANL: track 46.7 -> 54.1 mm
- net Net-(U5-Vbus): track 11.4 -> 16.7 mm
- net /USART2_TX: track 21.6 -> 16.3 mm
- net /USART2_RX: track 22.4 -> 17.2 mm, vias 2 -> 0
- net Net-(Q3-G): track 0.00 -> 4.89 mm
- net Net-(U7-IN): track 8.66 -> 12.5 mm
- net VBat: track 32.5 -> 36.2 mm
- net Net-(U6-IN): track 7.83 -> 11.5 mm
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Other:
- board text added: "3V3 GND VIN"
- board text added: "3V3 RST"
- board text added: "5V GND VIN"
- board text added: "CLK 3V3 GND"
- board text added: "CLK SWD"
- board text added: "GND GND"
- board text added: "GND V+"
- board text added: "MCU"
- board text added: "NTC"
- board text added: "RAK3172"
- board text added: "RESET TIME"
- board text added: "SDA SCL GND 3V3"
- board text added: "SWD RST GND"
- board text added: "VITAL Vector Drive Sensor Core v1 Lucas Ngo"
