File: SensorCore_v1/untitled.kicad_sch (KiCad schematic)
At the start: 5 parts, among them J1 2x3 Pogo Header, U2 RAK3172-9-SM-I

Commit message: SensorCore v1.0 - Approved
Parts:
- U2: Digikey Part (none) -> RAK3172-9-SM-I
Connections:
- net Net-(U7-BOOT0): no longer names the net of R3.1, U2.21 (BOOT0)
- net unconnected-(U7-PA0-Pad29): no longer names the net of U2.29 (PA0)
- net unconnected-(U7-PA1-Pad6): no longer names the net of U2.6 (PA1)
- net unconnected-(U7-PA10/PIN_A3-Pad25): no longer names the net of U2.25 (PA10/PIN_A3)
- net unconnected-(U7-PA11/SDA-Pad10): no longer names the net of U2.10 (PA11/SDA)
- net unconnected-(U7-PA12/SCL-Pad9): no longer names the net of U2.9 (PA12/SCL)
- net unconnected-(U7-PA15/PIN_A4-Pad3): no longer names the net of U2.3 (PA15/PIN_A4)
- net unconnected-(U7-PA4/~{SPI1_SS}-Pad16): no longer names the net of U2.16 (PA4/~{SPI1_SS})
- net unconnected-(U7-PA5/SPI1_CLK-Pad15): no longer names the net of U2.15 (PA5/SPI1_CLK)
- net unconnected-(U7-PA6/SPI1_MISO-Pad14): no longer names the net of U2.14 (PA6/SPI1_MISO)
- net unconnected-(U7-PA7/SPI1_MOSI-Pad13): no longer names the net of U2.13 (PA7/SPI1_MOSI)
- net unconnected-(U7-PA8-Pad19): no longer names the net of U2.19 (PA8)
- net unconnected-(U7-PA9-Pad20): no longer names the net of U2.20 (PA9)
- net unconnected-(U7-PB12-Pad27): no longer names the net of U2.27 (PB12)
- net unconnected-(U7-PB2/PIN_A2-Pad26): no longer names the net of U2.26 (PB2/PIN_A2)
- net unconnected-(U7-PB3/PIN_A0-Pad32): no longer names the net of U2.32 (PB3/PIN_A0)
- net unconnected-(U7-PB4/PIN_A1-Pad31): no longer names the net of U2.31 (PB4/PIN_A1)
- net unconnected-(U7-PB5-Pad30): no longer names the net of U2.30 (PB5)
- net unconnected-(U7-RF-Pad12): no longer names the net of U2.12 (RF)
- net unconnected-(U7-UART2_RX/PA3-Pad1): no longer names the net of U2.1 (UART2_RX/PA3)
- net unconnected-(U7-UART2_TX/PA2-Pad2): no longer names the net of U2.2 (UART2_TX/PA2)
Other:
- moved on the sheet: R3
